File: board/board.kicad_pcb (KiCad board)
At the start: 2 copper layers, 21 x 13 mm, 1 part

Commit message: initial
Parts:
- added C3: 100nF, Capacitor_SMD:C_0603_1608Metric, F.Cu at (154.4, 97.2)
- added C4: 100nF, Capacitor_SMD:C_0603_1608Metric, F.Cu at (154.4, 98.8)
- added J1: 022_battery_cells, on_edge:on_edge_2x05_device, F.Cu at (140.0, 96.5)
- added J2: 022_battery_cells, on_edge:on_edge_2x05_host, F.Cu at (161.0, 96.5)
- added Q3: FS3402, Package_TO_SOT_SMD:SOT-23, F.Cu at (153.9, 94.4)
- added Q4: FS3402, Package_TO_SOT_SMD:SOT-23, F.Cu at (149.9, 94.4)
- added R2: 330R, Resistor_SMD:R_0603_1608Metric, F.Cu at (151.2, 100.8)
- added R3: 330R, Resistor_SMD:R_0603_1608Metric, F.Cu at (154.4, 100.4)
- added R4: 2K, Resistor_SMD:R_0603_1608Metric, F.Cu at (146.8, 99.1)
- added U3: HY2120-CB, Package_TO_SOT_SMD:SOT-23-6, F.Cu at (150.5, 98.2)
- LOGO1: moved to B.Cu
- moved LOGO1 3.21 mm to (149.2, 95.9), turned to 180 degrees
Routing:
- net /protector/PB-: track 0.00 -> 22.0 mm
- net /protector/BAL: track 0.00 -> 21.9 mm, vias 0 -> 2
- net GND: track 0.00 -> 21.5 mm, vias 0 -> 24
- net /protector/PB+: track 0.00 -> 19.3 mm
- net Net-(J1-C3+4-): track 0.00 -> 17.8 mm
- net Net-(J1-C4+): track 0.00 -> 16.8 mm
- net Net-(Q3-G): track 0.00 -> 7.61 mm, vias 0 -> 2
- net Net-(Q4-G): track 0.00 -> 6.74 mm, vias 0 -> 2
- net Net-(U3-VDD): track 0.00 -> 6.28 mm
- net Net-(Q3-D): track 0.00 -> 4.00 mm
- net Net-(U3-VC): track 0.00 -> 3.69 mm
- net Net-(U3-CS): track 0.00 -> 1.72 mm
- added copper zone on B.Cu, net GND
- added copper zone on F.Cu, net GND
Other:
- outline, holes or cut-outs redrawn
