File: board/board.kicad_sch (KiCad schematic)
At the start: 1 part

Commit message: initial
Parts:
- added J1: 022_battery_cells, on_edge:on_edge_2x05_device, symbol put_on_edge:022_battery_cells
- added J2: 022_battery_cells, on_edge:on_edge_2x05_host, symbol put_on_edge:022_battery_cells
Connections:
- net GND: now also J1.1 (GND), J2.1 (GND)
- new net: J1.5 (C3+4-), J2.5 (C3+4-)
- new net: J1.6 (C4+), J2.6 (C4+)
- new net protector/BAL: J1.3 (C1+C2-), J2.3 (C1+C2-)
- new net protector/PB+: J1.4 (C2+C3-), J2.4 (C2+C3-)
- new net protector/PB-: J1.2 (C1-), J2.2 (C1-)
Other:
- sheet implementation renamed protector
- sheet protector: file implementation.kicad_sch -> protector.kicad_sch
- sheet protector ports: added BAL, PB+, PB-; removed none
- note removed: "Input connectors go here"
- note removed: "Output connectors go here"
